File: HW/KiCad/ts.kicad_pcb (KiCad board)
At the start: 2 copper layers, 80 x 45 mm, 45 parts, among them J1 AVR-ISP-6, J2 Conn_01x04, J3 Conn_01x04, J4 Conn_01x07, J5 Conn_01x04, J6 Conn_01x08, Q1 IRLZ34N, Q2 IRLZ34N, SW1 RESET, U1 ATmega328P-PU, U2 LM2576HVT-5, U3 HT7533, U4 LM75C, U5 4050, X1 Screw_Terminal_01x02, X2 Screw_Terminal_01x02, Y1 20MHz

Commit message: [HW] Add some layout
Routing:
- net +3V3: track 0.00 -> 38.9 mm, vias 0 -> 1
- net Net-(D1-Pad1): track 0.00 -> 37.0 mm
- net VCC: track 0.00 -> 18.6 mm
- net /LCD_NRST: track 0.00 -> 15.7 mm
- net /LCD_SCE: track 0.00 -> 12.7 mm
- added copper zone on B.Cu, net +12V
- added copper zone on F.Cu, net +12V
- added copper zone on B.Cu, net GND
- added copper zone on F.Cu, net GND
- added copper zone on F.Cu, net VCC
